File: adau_1701.kicad_sch (KiCad schematic)
At the start: 31 parts, among them J10 Conn_01x02_Pin, J9 Conn_01x04_Pin, U6 ADAU1701, U7 24LC256, Y1 12.288 MHz

Commit message: WIP: Converting to schematic
Parts:
- removed J10: Conn_01x02_Pin, symbol Connector:Conn_01x02_Pin
- removed J9: Conn_01x04_Pin, symbol Connector:Conn_01x04_Pin
- added C57: 100nF, Capacitor_SMD:C_0805_2012Metric_Pad1.18x1.45mm_HandSolder, symbol Device:C
- added J11, J12, J13: Conn_01x04_Pin, Connector_PinHeader_2.54mm:PinHeader_1x04_P2.54mm_Vertical, symbol Connector:Conn_01x04_Pin
- added J7: Conn_02x04_Odd_Even, Connector_PinHeader_2.54mm:PinHeader_2x04_P2.54mm_Vertical, symbol Connector_Generic:Conn_02x04_Odd_Even
- U7: footprint (none) -> Package_SO:SOIC-8_3.9x4.9mm_P1.27mm
- Y1: footprint Crystal:Crystal_SMD_7050-4Pin_7.0x5.0mm -> balanced-receiver:Crystal_SMD_7050-4Pin_7.0x5.0mm
- renumbered C19 to C23, C20 to C24, C21 to C25, C22 to C26, C33 to C27, C29 to C28, C40 to C29, C35 to C30, C25 to C31, C36 to C32, C26 to C33, C37 to C34, C39 to C35, C38 to C36, C27 to C37, C23 to C38, C28 to C39, C24 to C40, R10 to R11, R17 to R13, R13 to R15, R19 to R16, R20 to R17, R21 to R18
Connections:
- net +3.3V: now also C57.1, J12.1 (Pin_1), J12.2 (Pin_2), J12.3 (Pin_3), J12.4 (Pin_4)
- net +5V: now also J7.4 (Pin_4), J7.5 (Pin_5)
- net GND: now also C57.2, J13.1 (Pin_1), J13.2 (Pin_2), J13.3 (Pin_3), J13.4 (Pin_4), J7.2 (Pin_2), J7.7 (Pin_7), J7.8 (Pin_8)
- net MCLKI: now also Y1.4; no longer Y1.1
- net SCL: now also J7.1 (Pin_1)
- net SDA: now also J7.3 (Pin_3)
- net WP: now also J7.6 (Pin_6)
- net at C23.2, R11.2: now also Y1.1; no longer Y1.4
- net MP9: now reaches U6.26 (MP9)
- net MP9: now also J11.4 (Pin_4)
- net MP8: now reaches U6.27 (MP8)
- net MP8: now also J11.3 (Pin_3)
- net MP3: now reaches U6.28 (MP3)
- net MP3: now also J11.2 (Pin_2)
- net MP2: now reaches U6.29 (MP2)
- net MP2: now also J11.1 (Pin_1)
- no-connect marks 0 -> 8
Other:
- moved on the sheet: Y1

Commit message: WIP
Parts:
- removed C29: 100nF, Capacitor_SMD:C_0805_2012Metric_Pad1.18x1.45mm_HandSolder, symbol Device:C
- removed C39: 10uF, Capacitor_SMD:C_0805_2012Metric_Pad1.18x1.45mm_HandSolder, symbol Device:C
- removed Y1: 12.288 MHz, balanced-receiver:Crystal_SMD_7050-4Pin_7.0x5.0mm, symbol Device:Crystal_GND23
- added C62: 100nF, Capacitor_SMD:C_0805_2012Metric_Pad1.18x1.45mm_HandSolder, symbol Device:C
- added C9: 47uF, Capacitor_SMD:CP_Elec_5x5.4, symbol Device:C_Polarized
- added Q2: PNP, Package_TO_SOT_SMD:SOT-23, symbol Simulation_SPICE:PNP
- added R14: 1kΩ, Resistor_SMD:R_0805_2012Metric_Pad1.20x1.40mm_HandSolder, symbol Device:R
- added R37: 18kΩ, Resistor_SMD:R_0805_2012Metric_Pad1.20x1.40mm_HandSolder, symbol Device:R
- added Y2: 12.288MHz, Crystal:Crystal_SMD_3225-4Pin_3.2x2.5mm, symbol Device:Crystal_GND24
- C27: value 10uF -> 100nF
- R11: renamed from R14; value 7kΩ -> 18kΩ
- renumbered C57 to C41, J7 to J5, J12 to J6, J11 to J7, J13 to J8, R13 to R10, R15 to R12, R16 to R13, R17 to R15, R18 to R16, R11 to R8, R12 to R9, U6 to U5, U7 to U6
Connections:
- net +1.8V: now also C62.2, Q2.1 (C)
- net +3.3V: now also Q2.3 (E), R14.1
- net GND: now also C62.1, C9.2, R37.2, Y2.2, Y2.4; no longer U5.17 (VDRIVE)
- net MCLKI: now also Y2.3
- net at C23.2, R8.2: now also Y2.1
- net at U5.4 (ADC1): now also R37.1
- net at C37.2, U5.40 (CM): now also C9.1
- new net VDRIVE: Q2.2 (B), R14.2, U5.17 (VDRIVE)
Other:
- moved on the sheet: C36

Commit message: Completed PCB
Parts:
- added C39: 100nF, Capacitor_SMD:C_0805_2012Metric_Pad1.18x1.45mm_HandSolder, symbol Device:C
- added J12: Conn_01x02_Pin, Connector_PinHeader_2.54mm:PinHeader_1x02_P2.54mm_Vertical, symbol Connector:Conn_01x02_Pin
- added Q5, Q6: PMOS, Package_TO_SOT_SMD:SOT-23, symbol Simulation_SPICE:PMOS
- added R42, R43, R45, R46: 10k, Resistor_SMD:R_0805_2012Metric_Pad1.20x1.40mm_HandSolder, symbol Device:R
- added R44: 47k, Resistor_SMD:R_0805_2012Metric_Pad1.20x1.40mm_HandSolder, symbol Device:R
Connections:
- net +3.3V: now also R43.1, R45.1
- net +5V: now also R42.1
- net GND: now also C39.1, Q5.3 (S), Q6.3 (S)
- net MP4: now reaches U5.8 (MP4)
- net MP4: now also Q5.2 (G), R43.2
- net MP5: now reaches U5.9 (MP5)
- net MP5: now also Q6.2 (G), R45.2
- new net: Q5.1 (D), R42.2, R44.1
- new net MP4_5V: C39.2, J12.2 (Pin_2), R44.2
- new net MP5_VCC: J12.1 (Pin_1), Q6.1 (D), R46.2
- new net VCC: R46.1
- no-connect marks 8 -> 6
Other:
- company: (none) -> ${TITLE_BLOCK_AUTHOR}
- title: (none) -> ${TITLE_BLOCK_PROJECT_NAME}
- moved on the sheet: C23, C24, C41, J6, J7, J8, Q2, R13, R14, R15, R16, R8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
