File: analog_input.kicad_sch (KiCad schematic)
At the start: 12 parts, among them J1 NC3FAH2, U1 THAT1240

Commit message: WIP: Converting to schematic
Parts:
- removed TP1: Audio+, TestPoint:TestPoint_Pad_D1.0mm, symbol Connector:TestPoint
- removed TP2: Audio-, TestPoint:TestPoint_Pad_D1.0mm, symbol Connector:TestPoint
- removed TP4: AudioOut, TestPoint:TestPoint_Pad_D1.0mm, symbol Connector:TestPoint
- C22: renamed from C10; value 10uF -> 1uF
- R10: renamed from R3; value 1kΩ -> 10kΩ
- renumbered C2 to C17, C3 to C18, C4 to C19, C7 to C20, C8 to C21, J1 to J6, U1 to U5
Connections:
- net +5V renamed +5V_ANALOG
Other:
- moved on the sheet: C17, C18, C19, C20, C21, C22, J6, R10, U5

Commit message: WIP
Parts:
- removed J6: NC3FAH2, balanced-receiver:Jack_XLR_Neutrik_NC3FAH2_Horizontal, symbol Connector_Audio:NC3FAH2
- added J3: Conn_01x03_Pin, Connector_JST:JST_XH_B3B-XH-A_1x03_P2.50mm_Vertical, symbol Connector:Conn_01x03_Pin
- added J4: Conn_01x02_Pin, Connector_JST:JST_XH_B2B-XH-A_1x02_P2.50mm_Vertical, symbol Connector:Conn_01x02_Pin
- renumbered R10 to R7, U5 to U4
Connections:
- net Audio+: now also J3.1 (Pin_1)
- net Audio-: now also J3.3 (Pin_3)
- net GND: now also J3.2 (Pin_2), J4.2 (Pin_2)
- net Audio: now reaches C22.1, U4.5 (SNS), U4.6 (Vout)
- net Audio: now also J4.1 (Pin_1)
- net +5V_ANALOG renamed +5V

Commit message: Completed PCB
Other:
- company: (none) -> ${TITLE_BLOCK_AUTHOR}
- title: (none) -> ${TITLE_BLOCK_PROJECT_NAME}
Changed lines of the file:
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@@
 	(generator_version "9.0")
 	(paper "A4")
+	(title_block
+		(title "${TITLE_BLOCK_PROJECT_NAME}")
+		(date "${TITLE_BLOCK_DATE}")
+		(rev "${TITLE_BLOCK_REVISION}")
+		(company "${TITLE_BLOCK_AUTHOR}")
+		(comment 1 "${TITLE_BLOCK_REPOSITORY}")
+		(comment 8 "${TITLE_BLOCK_PROJECT_NAME_SHORT}")
+		(comment 9 "${TITLE_BLOCK_BASE_REPOSITORY}")
+	)
 	(junction
 		(at 163.83 115.57)
@@
 	)
 	(junction
-		(at 121.92 95.25)
-		(diameter 0)
-		(color 0 0 0 0)
-	)
-	(junction
 		(at 163.83 74.93)
 		(diameter 0)
@@
 	(wire
 		(pts
-			(xy 118.11 93.98) (xy 118.11 95.25)
-		)
-		(stroke
-			(width 0)
-			(type default)
-		)
-	)
-	(wire
-		(pts
 			(xy 163.83 74.93) (xy 161.29 74.93)
 		)
@@
 		(pts
 			(xy 121.92 95.25) (xy 121.92 97.79)
-		)
-		(stroke
-			(width 0)
-			(type default)
-		)
-	)
-	(wire
-		(pts
-			(xy 118.11 95.25) (xy 121.92 95.25)
 		)
 		(stroke
@@
 					(unit 1)
 				)
-			)
-		)
-	)
-	(symbol
-		(lib_id "power:PWR_FLAG")
-		(at 118.11 93.98 0)
-		(unit 1)
-		(exclude_from_sim no)
-		(in_bom yes)
-		(on_board yes)
-		(dnp no)
-		(fields_autoplaced yes)
-		(property "Reference" "#FLG01"
-			(at 118.11 92.075 0)
-			(effects
-				(font
-					(size 1.27 1.27)
-				)
-				(hide yes)
-			)
-		)
-		(property "Value" "PWR_FLAG"
-			(at 118.11 88.9 0)
-			(effects
-				(font
-					(size 1.27 1.27)
-				)
-			)
-		)
-		(property "Footprint" ""
-			(at 118.11 93.98 0)
-			(effects
-				(font
-					(size 1.27 1.27)
-				)
-				(hide yes)
-			)
-		)
-		(property "Datasheet" "~"
-			(at 118.11 93.98 0)
-			(effects
-				(font
-					(size 1.27 1.27)
-				)
-				(hide yes)
-			)
-		)
-		(property "Description" "Special symbol for telling ERC where power comes from"
-			(at 118.11 93.98 0)
-			(effects
-				(font
-					(size 1.27 1.27)
-				)
-				(hide yes)
-			)
-		)
-		(pin "1"
-		)
-		(instances
-			(project "balanced-receiver"
-				(path "/6a415962-4bc6-46b3-a4a9-4a4125d0fb6a/a2301bca-fb76-48bf-8387-0002b51351ca"
-					(reference "#FLG01")
-					(unit 1)
-				)
