File: analog_output.kicad_sch (KiCad schematic)
At the start: 40 parts, among them J11 Conn_01x03_Pin, J12 Conn_01x03_Pin, U4 OPA1612AxD, U5 OPA1612AxD

Commit message: WIP: Converting to schematic
Parts:
- added C60, C61, C62, C63: 10uF, Capacitor_SMD:C_0805_2012Metric_Pad1.18x1.45mm_HandSolder, symbol Device:C
- J10: renamed from J12; footprint (none) -> Connector_JST:JST_XH_B3B-XH-A_1x03_P2.50mm_Vertical
- J9: renamed from J11; footprint Connector_Hirose:Hirose_DF13-03P-1.25DS_1x03_P1.25mm_Horizontal -> Connector_JST:JST_XH_B3B-XH-A_1x03_P2.50mm_Vertical
- U8: renamed from U4; footprint (none) -> Package_SO:SOIC-8_3.9x4.9mm_P1.27mm
- U9: renamed from U5; footprint (none) -> Package_SO:SOIC-8_3.9x4.9mm_P1.27mm
- renumbered C46 to C42, C47 to C44, C42 to C45, C48 to C46, C55 to C47, C56 to C48, C44 to C49, C45 to C50, C49 to C51, C50 to C53, C53 to C54, C51 to C55, C54 to C56, R11 to R19, R23 to R20, R15 to R21, R24 to R22, R16 to R23, R25 to R24, R22 to R25, R18 to R27, R27 to R28, R28 to R29, R33 to R30, R29 to R31, R34 to R32, R30 to R33, R35 to R34, R31 to R35, R32 to R37, R37 to R38
Connections:
- net -5V: now also C61.1, C62.1
- net ADAU_AUDIO_OUTPUT_0: now also C51.1; no longer C41.1
- net ADAU_AUDIO_OUTPUT_1: now also C41.1; no longer C42.1
- net ADAU_AUDIO_OUTPUT_2: now also C42.1; no longer C51.1
- net AUDIO_OUT_0: now also J10.3 (Pin_3); no longer J9.3 (Pin_3)
- net AUDIO_OUT_1: now also J9.3 (Pin_3); no longer J9.1 (Pin_1)
- net AUDIO_OUT_2: now also J10.1 (Pin_1); no longer J10.3 (Pin_3)
- net AUDIO_OUT_3: now also J9.1 (Pin_1); no longer J10.1 (Pin_1)
- net GND: now also C60.2, C61.2, C62.2, C63.2
- net +5V renamed +5V_ANALOG
- net +5V_ANALOG: now also C60.1, C63.1
Other:
- moved on the sheet: C47, C48, C49, C50, U8C, U9C

Commit message: WIP
Parts:
- removed C42, C51, C52: 1uF, Capacitor_SMD:C_0805_2012Metric_Pad1.18x1.45mm_HandSolder, symbol Device:C
- removed R20, R29, R30: 10kΩ, Resistor_SMD:R_0805_2012Metric_Pad1.20x1.40mm_HandSolder, symbol Device:R
- added C47, C60, C61: 1uF, Capacitor_SMD:C_0805_2012Metric_Pad1.18x1.45mm_HandSolder, symbol Device:C
- added R26, R35, R36: 10kΩ, Resistor_SMD:R_0805_2012Metric_Pad1.20x1.40mm_HandSolder, symbol Device:R
- renumbered C43 to C42, C44 to C43, C45 to C44, C46 to C45, C41 to C46, C60 to C48, C47 to C49, C48 to C50, C61 to C51, C63 to C52, C49 to C53, C50 to C54, C62 to C55, C53 to C56, C54 to C57, C55 to C58, C56 to C59, R21 to R17, R22 to R18, R23 to R19, R24 to R20, R25 to R21, R26 to R22, R27 to R23, R28 to R24, R19 to R25, R31 to R27, R32 to R28, R33 to R29, R34 to R30, R35 to R31, R36 to R32, R37 to R33, R38 to R34, U8 to U7, U9 to U8
Connections:
- net ADAU_AUDIO_OUTPUT_0: now also R17.1
- net ADAU_AUDIO_OUTPUT_1: now also R18.1; no longer C46.1
- net ADAU_AUDIO_OUTPUT_2: now also R27.1
- net ADAU_AUDIO_OUTPUT_3: now also R28.1
- net AUDIO_OUT_0: now also C46.2, J9.3 (Pin_3), R25.1; no longer C44.2, J10.3 (Pin_3), R23.2, U7.1
- net AUDIO_OUT_1: now also J9.1 (Pin_1), C47.2, R26.1; no longer C45.2, J9.3 (Pin_3), R24.2, U7.7
- net AUDIO_OUT_2: now also C60.2, R35.1; no longer C58.2, R33.2, U8.1
- net AUDIO_OUT_3: now also J10.3 (Pin_3), C61.2, R36.1; no longer C59.2, J9.1 (Pin_1), R34.2, U8.7
- net GND: now also R26.2, R35.2, R36.2
- net +5V_ANALOG renamed +5V
- new net: C44.2, C46.1, R23.2, U7.1
- new net: C45.2, C47.1, R24.2, U7.7
- new net: C58.2, C60.1, R33.2, U8.1
- new net: C59.2, C61.1, R34.2, U8.7
Other:
- moved on the sheet: C42, C43, C44, C45, C46, C48, C49, C50, C51, C52, C53, C54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

Commit message: Completed PCB
Other:
- company: (none) -> ${TITLE_BLOCK_AUTHOR}
- title: (none) -> ${TITLE_BLOCK_PROJECT_NAME}
Changed lines of the file:
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@@
 	(generator_version "9.0")
 	(paper "A4")
+	(title_block
+		(title "${TITLE_BLOCK_PROJECT_NAME}")
+		(date "${TITLE_BLOCK_DATE}")
+		(rev "${TITLE_BLOCK_REVISION}")
+		(company "${TITLE_BLOCK_AUTHOR}")
+		(comment 1 "${TITLE_BLOCK_REPOSITORY}")
+		(comment 8 "${TITLE_BLOCK_PROJECT_NAME_SHORT}")
+		(comment 9 "${TITLE_BLOCK_BASE_REPOSITORY}")
+	)
 	(junction
 		(at 240.03 107.95)
