File: balanced-receiver.kicad_pcb (KiCad board)
At the start: 2 copper layers, 55.5 x 89 mm, 131 parts, among them J1 Barrel_Jack_Switch, J10 Conn_01x03_Pin, J11 Conn_01x04_Pin, J12 Conn_01x04_Pin, J13 Conn_01x04_Pin, J2 Screw_Terminal_01x02, J3 Screw_Terminal_01x02, J4 Screw_Terminal_01x03, J6 NC3FAH2, J7 Conn_02x04_Odd_Even, J9 Conn_01x03_Pin, Q1 Q_PMOS_GDS, U1 LM1117DT-3.3, U2 LM1117DT-1.8, U3 TPS62932, U4 LM2776, U5 THAT1240, U6 ADAU1701, U7 24LC256, U8 OPA1612AxD, U9 OPA1612AxD, Y1 12.288 MHz

Commit message: WIP
Parts:
- removed C10, C29: 100nF, Capacitor_SMD:C_0805_2012Metric_Pad1.18x1.45mm_HandSolder
- removed the C15 at (58.9, 111.9)
- removed the C16 at (55.4, 96.3)
- removed C39: 10uF, Capacitor_SMD:C_0805_2012Metric_Pad1.18x1.45mm_HandSolder
- removed the C42 at (63.9, 57.3)
- removed the C51 at (28.9, 50.5)
- removed the C52 at (63.9, 46.0)
- removed the C58 at (55.4, 88.6)
- removed the C59 at (55.4, 90.9)
- removed the J2 at (77.0, 114.9)
- removed the J6 at (38.2, 94.4)
- removed the R1 at (48.1, 95.8)
- removed the R20 at (60.9, 57.3)
- removed the R29 at (31.9, 50.5)
- removed the R30 at (60.9, 46.0)
- removed REF** (x4): MountingHole_2.2mm_M2_DIN965_Pad, MountingHole:MountingHole_2.2mm_M2_DIN965_Pad
- removed TP2: VCC_P, TestPoint:TestPoint_Pad_D1.0mm
- removed the U3 at (54.8, 100.8)
- removed the U4 at (54.6, 100.8)
- removed Y1: 12.288 MHz, balanced-receiver:Crystal_SMD_7050-4Pin_7.0x5.0mm
- added C2: 10uF, Capacitor_SMD:C_0805_2012Metric_Pad1.18x1.45mm_HandSolder, F.Cu at (57.6, 69.7)
- added C47: 1uF, Capacitor_SMD:C_0805_2012Metric_Pad1.18x1.45mm_HandSolder, F.Cu at (44.0, 20.0)
- added C6: 10nF, Capacitor_SMD:C_0805_2012Metric_Pad1.18x1.45mm_HandSolder, F.Cu at (52.4, 82.3)
- added C60: 1uF, Capacitor_SMD:C_0805_2012Metric_Pad1.18x1.45mm_HandSolder, F.Cu at (58.7, 20.2)
- added C61: 1uF, Capacitor_SMD:C_0805_2012Metric_Pad1.18x1.45mm_HandSolder, F.Cu at (70.1, 20.2)
- added C62: 100nF, Capacitor_SMD:C_0805_2012Metric_Pad1.18x1.45mm_HandSolder, F.Cu at (53.5, 57.1)
- added D2: B340A, Diode_SMD:D_SMA_Handsoldering, F.Cu at (30.5, 75.0)
- added D3: B340A, Diode_SMD:D_SMA_Handsoldering, F.Cu at (53.6, 75.0)
- added H1: MountingHole_Pad_MP, MountingHole:MountingHole_2.2mm_M2_DIN965_Pad_TopBottom, F.Cu at (27.1, 86.4)
- added H2: MountingHole_Pad_MP, MountingHole:MountingHole_2.2mm_M2_DIN965_Pad_TopBottom, F.Cu at (85.1, 86.4)
- added H3: MountingHole_Pad_MP, MountingHole:MountingHole_2.2mm_M2_DIN965_Pad_TopBottom, F.Cu at (85.1, 17.4)
- added H4: MountingHole_Pad_MP, MountingHole:MountingHole_2.2mm_M2_DIN965_Pad_TopBottom, F.Cu at (27.1, 17.4)
- added J3: Conn_01x03_Pin, Connector_JST:JST_XH_B3B-XH-A_1x03_P2.50mm_Vertical, F.Cu at (27.1, 40.9)
- added L4: 1uH, Inductor_SMD:L_APV_APH0420, F.Cu at (70.1, 74.1)
- added Q2: PNP, Package_TO_SOT_SMD:SOT-23, F.Cu at (58.2, 62.4)
- added R14: 1kΩ, Resistor_SMD:R_0805_2012Metric_Pad1.20x1.40mm_HandSolder, F.Cu at (55.3, 62.3)
- added R26: 10kΩ, Resistor_SMD:R_0805_2012Metric_Pad1.20x1.40mm_HandSolder, F.Cu at (44.0, 17.8)
- added R35: 10kΩ, Resistor_SMD:R_0805_2012Metric_Pad1.20x1.40mm_HandSolder, F.Cu at (58.7, 18.0)
- added R36: 10kΩ, Resistor_SMD:R_0805_2012Metric_Pad1.20x1.40mm_HandSolder, F.Cu at (70.0, 18.0)
- added R37: 18kΩ, Resistor_SMD:R_0805_2012Metric_Pad1.20x1.40mm_HandSolder, F.Cu at (50.2, 53.8)
- added R4: 10kΩ, Resistor_SMD:R_0805_2012Metric_Pad1.20x1.40mm_HandSolder, F.Cu at (62.3, 82.7)
- added U1: TPS5430DDA, Package_SO:TI_SO-PowerPAD-8, F.Cu at (35.4, 77.6)
- added Y2: 12.288MHz, Crystal:Crystal_SMD_3225-4Pin_3.2x2.5mm, F.Cu at (69.9, 54.8)
- C11: value 1uF -> 22pF; moved to F.Cu
- C12: value 100nF -> 22pF
- C15: renamed from C2; moved to F.Cu
- C16: renamed from C6; moved to F.Cu
- C17, C18, C19, C3, C30, C31, C32, C33, C34, C35, C36, C37, C38, C40, D1, F1, Q1: moved to F.Cu
- C27: value 10uF -> 100nF; moved to F.Cu
- C48: renamed from C60; moved to F.Cu
- C49: renamed from C47; moved to F.Cu
- C5: value 100nF -> 10nF
- C50: renamed from C48; moved to F.Cu
- C51: renamed from C61; moved to F.Cu
- C52: renamed from C63; moved to F.Cu
- C53: renamed from C49; moved to F.Cu
- C54: renamed from C50; moved to F.Cu
- C55: renamed from C62; moved to F.Cu
- C7: value 10uF -> 220uF; footprint Capacitor_SMD:C_0805_2012Metric_Pad1.18x1.45mm_HandSolder -> Capacitor_SMD:CP_Elec_6.3x7.7; moved to F.Cu
- C8: value 33nF -> 220uF; footprint Capacitor_SMD:C_0805_2012Metric_Pad1.18x1.45mm_HandSolder -> Capacitor_SMD:CP_Elec_6.3x7.7
- C9: value 2.2uF -> 47uF; footprint Capacitor_SMD:C_0805_2012Metric_Pad1.18x1.45mm_HandSolder -> Capacitor_SMD:CP_Elec_5x5.4; moved to F.Cu
- J1: value Barrel_Jack_Switch -> Power; footprint balanced-receiver:BarrelJack_GCT_DCJ200-10-A_Horizontal -> Connector_JST:JST_XH_B2B-XH-A_1x02_P2.50mm_Vertical
- J4: value Screw_Terminal_01x03 -> Conn_01x02_Pin; footprint balanced-receiver:TerminalBlock_1x03_P7.50mm_Horizontal -> Connector_JST:JST_XH_B2B-XH-A_1x02_P2.50mm_Vertical
- L1: value 6.8uH -> 22uH; footprint Inductor_SMD:L_APV_APH0530 -> Inductor_SMD:L_APV_ANR6028
- L2: value 1uH -> 22uH; footprint Inductor_SMD:L_0805_2012Metric_Pad1.05x1.20mm_HandSolder -> Inductor_SMD:L_APV_ANR6028; moved to F.Cu
- L3: footprint Inductor_SMD:L_0805_2012Metric_Pad1.05x1.20mm_HandSolder -> Inductor_SMD:L_APV_APH0420; moved to F.Cu
- R1: renamed from R4; moved to F.Cu
- R11: renamed from R14; value 7kΩ -> 18kΩ
- R2: value 91kΩ -> 10kΩ
- R3: value 9.1kΩ -> 3.3k
- R5: value 47kΩ -> 3.3kΩ
- R6: renamed from R7; moved to F.Cu
- U2: value LM1117DT-1.8 -> TPS5430DDA; footprint Package_TO_SOT_SMD:SOT-223-3_TabPin2 -> Package_SO:TI_SO-PowerPAD-8; moved to F.Cu
- U3: renamed from U1; moved to F.Cu
- moved R6 71.1 mm to (29.2, 55.3), turned to 0 degrees
- moved D4 69.3 mm to (29.2, 57.5), turned to 0 degrees
- moved C9 66.8 mm to (64.1, 37.7), turned to 0 degrees
- moved J4 52.9 mm to (27.1, 49.9), turned to 90 degrees
- moved C19 49.5 mm to (43.8, 43.4), turned to 0 degrees
- moved J1 47.3 mm to (27.1, 64.4), turned to 90 degrees
- moved D1 45.8 mm to (37.1, 59.5), turned to 180 degrees
- moved C17 45.4 mm to (40.7, 44.2), turned to 90 degrees
- moved C21 45.2 mm to (44.5, 38.9), turned to 90 degrees
- moved R1 44.1 mm to (36.6, 62.0), turned to 0 degrees
- moved R25 43.9 mm to (32.7, 17.9), turned to 0 degrees
- moved C18 43.0 mm to (37.5, 43.4)
- moved C20 42.3 mm to (36.7, 38.2), turned to -90 degrees
- moved F1 42.1 mm to (42.0, 64.8)
- moved C46 41.8 mm to (32.7, 20.1), turned to 180 degrees
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- renumbered C57 to C41, C43 to C42, C44 to C43, C45 to C44, C46 to C45, C41 to C46, C53 to C56, C54 to C57, C55 to C58, C56 to C59, D2 to D4, J3 to J2, J7 to J5, J12 to J6, J11 to J7, J13 to J8, R13 to R10, R15 to R12, R16 to R13, R17 to R15, R18 to R16, R21 to R17, R22 to R18, R23 to R19, R24 to R20, R25 to R21, R26 to R22, R27 to R23, R28 to R24, R19 to R25, R31 to R27, R32 to R28, R33 to R29, R34 to R30, R35 to R31, R36 to R32, R37 to R33, R38 to R34, R10 to R7, R11 to R8, R12 to R9, U5 to U4, U6 to U5, U7 to U6, U8 to U7, U9 to U8
Connections:
- C1 pad 1: VCC_P -> VCC
- C11 pad 1: Net-(U4-C1+) -> Net-(C11-Pad1)
- C11 pad 2: Net-(U4-C1-) -> Net-(U1-VSENSE)
- C12 pad 1: Net-(U3-FB) -> GND
- C12 pad 2: +5V -> Net-(U2-VSENSE)
- C14 pad 1: +5V -> GND
- C14 pad 2: GND -> -5V
- C20 pad 1: +5V_ANALOG -> +5V
- C22 pad 1: Net-(U5-SNS) -> /analog_input/Audio
- C3 pad 1: GND -> VCC
- C3 pad 2: +5V -> GND
- C37 pad 2: Net-(U6-CM) -> Net-(U5-CM)
- C4 pad 1: VCC_P -> VCC
- C4 pad 2: GND -> Net-(D3-A)
- C44 pad 2: /analog_output/AUDIO_OUT_0 -> Net-(C44-Pad2)
- C45 pad 2: /analog_output/AUDIO_OUT_1 -> Net-(C45-Pad2)
- C46 pad 1: ADAU_AUDIO_OUTPUT_1 -> Net-(C44-Pad2)
- C46 pad 2: Net-(C41-Pad2) -> /analog_output/AUDIO_OUT_0
- C48 pad 1: +5V_ANALOG -> +5V
- C49 pad 1: +5V_ANALOG -> +5V
- C5 pad 1: VCC_P -> Net-(U1-BOOT)
- C5 pad 2: GND -> Net-(D2-K)
- C52 pad 1: +5V_ANALOG -> +5V
- C53 pad 1: +5V_ANALOG -> +5V
- C58 pad 2: /analog_output/AUDIO_OUT_2 -> Net-(C58-Pad2)
- C59 pad 2: /analog_output/AUDIO_OUT_3 -> Net-(C59-Pad2)
- C7 pad 1: GND -> Net-(C11-Pad1)
- C7 pad 2: +1.8V -> GND
- C8 pad 1: Net-(U3-SS) -> GND
- C8 pad 2: GND -> Net-(D3-A)
- C9 pad 1: +5V -> Net-(U5-CM)
- D4 pad 2: VCC_P -> VCC
- F1 pad 2: VCC_P -> VCC
- J1 pad 1: VCC_UN -> Net-(J1-Pin_1)
- J10 pad 3: /analog_output/AUDIO_OUT_0 -> /analog_output/AUDIO_OUT_3
- J4 pad 1: GND -> /analog_input/Audio
- J4 pad 2: VCC_UN -> GND
- J9 pad 1: /analog_output/AUDIO_OUT_3 -> /analog_output/AUDIO_OUT_1
- J9 pad 3: /analog_output/AUDIO_OUT_1 -> /analog_output/AUDIO_OUT_0
- L1 pad 1: Net-(U3-SW) -> Net-(D2-K)
- L1 pad 2: +5V -> Net-(C11-Pad1)
- L2 pad 1: +5V -> Net-(D3-K)
- L2 pad 2: +5V_ANALOG -> GND
- L3 pad 1: Net-(U4-VOUT) -> Net-(C11-Pad1)
- L3 pad 2: -5V -> +5V
- Q1 pad 2: VCC -> Net-(J1-Pin_1)
- R17 pad 1: Net-(C41-Pad2) -> ADAU_AUDIO_OUTPUT_0
- R18 pad 1: Net-(C42-Pad2) -> ADAU_AUDIO_OUTPUT_1
- R2 pad 1: Net-(U3-EN) -> Net-(U1-VSENSE)
- R2 pad 2: GND -> Net-(C11-Pad1)
- R23 pad 2: /analog_output/AUDIO_OUT_0 -> Net-(C44-Pad2)
- R24 pad 2: /analog_output/AUDIO_OUT_1 -> Net-(C45-Pad2)
- R25 pad 1: Net-(C41-Pad2) -> /analog_output/AUDIO_OUT_0
- R27 pad 1: Net-(C51-Pad2) -> ADAU_AUDIO_OUTPUT_2
- R28 pad 1: Net-(C52-Pad2) -> ADAU_AUDIO_OUTPUT_3
- R3 pad 1: Net-(U3-FB) -> Net-(U1-VSENSE)
- R33 pad 2: /analog_output/AUDIO_OUT_2 -> Net-(C58-Pad2)
- R34 pad 2: /analog_output/AUDIO_OUT_3 -> Net-(C59-Pad2)
- R5 pad 1: +5V -> Net-(U2-VSENSE)
- R5 pad 2: Net-(U3-FB) -> Net-(D3-A)
- U2 pad 1: GND -> Net-(U2-BOOT)
- U2 pad 2: +1.8V -> unconnected-(U2-NC-Pad2)
- U2 pad 3: +5V -> unconnected-(U2-NC-Pad3)
- U4 pad 5: Net-(U5-SNS) -> /analog_input/Audio
- U4 pad 6: Net-(U5-SNS) -> /analog_input/Audio
- U4 pad 7: +5V_ANALOG -> +5V
- U5 pad 17: GND -> /adau_1701/VDRIVE
- U5 pad 40: Net-(U6-CM) -> Net-(U5-CM)
- U7 pad 1: /analog_output/AUDIO_OUT_0 -> Net-(C44-Pad2)
- U7 pad 7: /analog_output/AUDIO_OUT_1 -> Net-(C45-Pad2)
- U7 pad 8: +5V_ANALOG -> +5V
- U8 pad 1: /analog_output/AUDIO_OUT_2 -> Net-(C58-Pad2)
- U8 pad 7: /analog_output/AUDIO_OUT_3 -> Net-(C59-Pad2)
- U8 pad 8: +5V_ANALOG -> +5V
Routing:
- net GND: track 2.65 -> 160.2 mm, vias 63 -> 56
- net +3.3V: track 175.0 -> 44.1 mm, vias 5 -> 14
- net +5V: track 143.6 -> 238.0 mm, vias 1 -> 7
- net +5V_ANALOG: track 87.1 -> 0.00 mm, vias 3 -> 0
- net VCC_P: track 72.1 -> 0.00 mm, vias 2 -> 0
- net VCC_UN: track 70.0 -> 0.00 mm
- net /analog_input/Audio: track 0.00 -> 35.9 mm
- net Net-(C11-Pad1): track 0.00 -> 34.0 mm
- net /analog_output/AUDIO_OUT_3: track 52.7 -> 20.6 mm, vias 1 -> 0
- net VCC: track 49.0 -> 18.6 mm, vias 1 -> 10
- net +1.8V: track 49.3 -> 19.2 mm, vias 3 -> 2
- net /analog_output/AUDIO_OUT_2: track 58.1 -> 33.8 mm, vias 1 -> 0
- net -5V: track 79.7 -> 103.8 mm, vias 3 -> 4
- net /adau_1701/WP: track 59.1 -> 36.0 mm, vias 2 -> 3
- net Net-(D2-K): track 0.00 -> 22.7 mm
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- added copper zone on F.Cu, net +3.3V
- added copper zone on In2.Cu, net +3.3V
- added copper zone on In1.Cu, net GND
- added copper zone on F.Cu, net Net-(D3-A)
- added copper zone on F.Cu, net VCC
- added copper zone on In2.Cu, net VCC
- removed copper zone on B.Cu, net GND
Other:
- board size 55.5 x 89 mm -> 65 x 76 mm
- copper layers 2 -> 4
- board text added: "INPUT A -"
- board text added: "INPUT A- - A+"
- board text added: "OUTPUT A0 - A1"
- board text added: "OUTPUT A2 - A3"
- board text added: "POWER + -"
- board text removed: "AMP SW + -"
- board text removed: "AUDIO A0 - A2"
- board text removed: "AUDIO A1 - A3"
- board text removed: "POWER SWITCH"
- board text removed: "PWR"
- board text removed: "{ "ViaStitching": "0.2", "stitch_zone_0": { "HSpacing": "5", "VSpacing": "5", "HOffset": "0", "VOffset": "0", "Clearance": "0", "Randomize": false } }"

Commit message: Completed PCB
Parts:
- added C39: 100nF, Capacitor_SMD:C_0805_2012Metric_Pad1.18x1.45mm_HandSolder, F.Cu at (127.8, 71.3)
- added J12: Conn_01x02_Pin, Connector_PinHeader_2.54mm:PinHeader_1x02_P2.54mm_Vertical, B.Cu at (135.7, 66.2)
- added Q5: PMOS, Package_TO_SOT_SMD:SOT-23, F.Cu at (122.6, 71.4)
- added Q6: PMOS, Package_TO_SOT_SMD:SOT-23, F.Cu at (122.7, 60.2)
- added R42: 10k, Resistor_SMD:R_0805_2012Metric_Pad1.20x1.40mm_HandSolder, F.Cu at (126.6, 74.3)
- added R43: 10k, Resistor_SMD:R_0805_2012Metric_Pad1.20x1.40mm_HandSolder, F.Cu at (122.6, 68.4)
- added R44: 47k, Resistor_SMD:R_0805_2012Metric_Pad1.20x1.40mm_HandSolder, F.Cu at (125.7, 71.3)
- added R45: 10k, Resistor_SMD:R_0805_2012Metric_Pad1.20x1.40mm_HandSolder, F.Cu at (122.6, 63.0)
- added R46: 10k, Resistor_SMD:R_0805_2012Metric_Pad1.20x1.40mm_HandSolder, F.Cu at (122.6, 57.3)
- moved J5 54.9 mm to (130.8, 79.3)
- moved J2 54.9 mm to (137.1, 87.4)
- moved H2 53.2 mm to (137.3, 96.5)
- moved H3 53.2 mm to (137.3, 27.5)
- moved J6 53.0 mm to (130.6, 58.0)
- moved J7 53.0 mm to (130.6, 60.5)
- moved J8 53.0 mm to (130.6, 55.4)
- moved J10 53.0 mm to (137.1, 33.4)
- moved J9 53.0 mm to (137.1, 44.9)
- moved C57 51.3 mm to (119.4, 37.5)
- moved C61 51.3 mm to (120.4, 30.2)
- moved R34 51.3 mm to (119.4, 33.5)
- moved U8 51.3 mm to (114.5, 35.8)
- moved C42 51.3 mm to (83.6, 37.2)
- moved C43 51.3 mm to (93.4, 37.2)
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Connections:
- U5 pad 8: unconnected-(U5-MP4-Pad8) -> /adau_1701/MP4
- U5 pad 9: unconnected-(U5-MP5-Pad9) -> /adau_1701/MP5
Routing:
- net VCC: track 18.6 -> 53.0 mm, vias 10 -> 12
- net /adau_1701/MP5: track 0.00 -> 29.4 mm, vias 0 -> 2
- net /adau_1701/MP4: track 0.00 -> 27.2 mm, vias 0 -> 2
- net /adau_1701/MP5_VCC: track 0.00 -> 22.6 mm
- net GND: track 160.2 -> 180.4 mm, vias 56 -> 61
- net +3.3V: track 44.1 -> 62.3 mm, vias 14 -> 16
- net +5V: track 238.0 -> 256.1 mm, vias 7 -> 8
- net /adau_1701/MP4_5V: track 0.00 -> 15.6 mm
- net /adau_1701/SDA: track 33.0 -> 41.2 mm
- net /adau_1701/MP3: track 23.5 -> 28.3 mm
- net /adau_1701/MP9: track 26.2 -> 30.9 mm
- net Net-(Q5-D): track 0.00 -> 4.56 mm
- net Net-(J1-Pin_1): track 9.31 -> 13.8 mm
- net /adau_1701/MP8: track 24.2 -> 27.8 mm
- net /adau_1701/MP2: track 22.6 -> 26.1 mm
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Other:
- board size 65 x 76 mm -> 70 x 76 mm
- board text added: "ENB"
- board text added: "MUTE"
